Commit message: add station and controller

File: crane_x7_manipulation/rsc/crane_x7_description/crane_x7.urdf (robot description, URDF)
Before this commit: robot crane_x7, 21 links, 20 joints
Joints:
- joint crane_x7_gripper_finger_a_joint: axis (none) -> 0 -1 0; limit (none) -> lower=0.0046 upper=1.62601 effort=4.0 velocity=4.81710873
- joint crane_x7_gripper_finger_b_joint: axis (none) -> 0 1 0; limit (none) -> lower=0.0046 upper=1.62601 effort=4.0 velocity=4.81710873
